Commit message: 加载nero但是训练效果差

File: src/isaac_so_arm101/robots/nero_description/urdf/nero_description_stand_v2.urdf (robot description, URDF)
Before this commit: robot nero_description, 10 links, 9 joints
Links:
- link base_link: geometry collision mesh filename=../meshes/base_link.STL; visual mesh filename=../meshes/dae/base_link.dae
- link end_effector: geometry collision mesh filename=../meshes/stand_v2.dae; visual mesh filename=../meshes/stand_v2.dae
- link link1: geometry collision mesh filename=../meshes/Link1.STL; visual mesh filename=../meshes/dae/link1.dae
- link link2: geometry collision mesh filename=../meshes/Link2.STL; visual mesh filename=../meshes/dae/link2.dae
- link link3: geometry collision mesh filename=../meshes/Link3.STL; visual mesh filename=../meshes/dae/link3.dae
- link link4: geometry collision mesh filename=../meshes/Link4.STL; visual mesh filename=../meshes/dae/link4.dae
- link link5: geometry collision mesh filename=../meshes/Link5.STL; visual mesh filename=../meshes/dae/link5.dae
- link link6: geometry collision mesh filename=../meshes/Link6.STL; visual mesh filename=../meshes/dae/link6.dae
- link link7: geometry collision mesh filename=../meshes/Link7.STL; visual mesh filename=../meshes/dae/link7.dae
- link world: mass None -> 0.77; geometry collision box size=0.01 0.01 0.01; visual box size=0.01 0.01 0.01
Joints:
- joint world_to_base_link: origin xyz=0 0 0 rpy=0 0 0 -> xyz=0 0 0 rpy=0 0 3.14

Commit message: 修改URDF

File: src/isaac_so_arm101/robots/nero_description/urdf/nero_description_stand_v2.urdf (robot description, URDF)
Before this commit: robot nero_description, 10 links, 9 joints
Links:
- removed link end_effector
- added link end_effector_link, mass 0.05; collision mesh filename=../meshes/stand_v2.dae; visual mesh filename=../meshes/stand_v2.dae
Joints:
- joint end_effector_joint: child end_effector -> end_effector_link
- joint world_to_base_link: origin xyz=0 0 0 rpy=0 0 3.14 -> xyz=0 0 0 rpy=0 0 0.0
