Commit message: 增加nero lift RL 案例

File: src/isaac_so_arm101/robots/nero_description/urdf/nero_description.urdf (robot description, URDF)
Before this commit: robot nero_description, 10 links, 9 joints
Links:
- removed link end_effector
- link base_link: mass 0.77 -> 1.06458435; geometry collision mesh filename=../meshes/base_link.stl; visual mesh filename=../meshes/dae/base_link.dae
- link link1: mass 0.77 -> 0.76710504; geometry collision mesh filename=../meshes/link1.stl; visual mesh filename=../meshes/dae/link1.dae
- link link2: mass 0.49 -> 0.69381908; geometry collision mesh filename=../meshes/link2.stl; visual mesh filename=../meshes/dae/link2.dae
- link link3: mass 0.67 -> 0.67246544; geometry collision mesh filename=../meshes/link3.stl; visual mesh filename=../meshes/dae/link3.dae
- link link4: mass 0.41 -> 0.48451414; geometry collision mesh filename=../meshes/link4.stl; visual mesh filename=../meshes/dae/link4.dae
- link link5: mass 0.56 -> 0.58368405; geometry collision mesh filename=../meshes/link5.stl; visual mesh filename=../meshes/dae/link5.dae
- link link6: mass 0.31 -> 0.3140406; geometry collision mesh filename=../meshes/link6.stl; visual mesh filename=../meshes/dae/link6.dae
- link link7: geometry collision mesh filename=../meshes/link7.stl; visual mesh filename=../meshes/dae/link7.dae
Joints:
- removed joint end_effector_joint
- joint joint1: limit lower=-2.7 upper=2.7 effort=0 velocity=0 -> lower=-2.70526 upper=2.70526 effort=100 velocity=5
- joint joint2: limit lower=-1.74 upper=1.74 effort=0 velocity=0 -> lower=-1.74 upper=1.74 effort=100 velocity=5; origin xyz=0 0 0 rpy=1.5708 3.1415 0 -> xyz=0 0 0 rpy=1.5707963  3.1415926 0
- joint joint3: limit lower=-2.75 upper=2.75 effort=0 velocity=0 -> lower=-2.75 upper=2.75 effort=100 velocity=5; origin xyz=0 -0.31 0 rpy=-1.5708 0 3.1416 -> xyz=0 -0.31 0 rpy=-1.5707963  0 3.1415926926
- joint joint4: limit lower=-1.01 upper=2.14 effort=0 velocity=0 -> lower=-1.01 upper=2.14 effort=100 velocity=5; origin xyz=0 0 0 rpy=-1.5708 0 3.1416 -> xyz=0 0 0 rpy=-1.5707963  0 3.1415926926
- joint joint5: limit lower=-2.75 upper=2.75 effort=0 velocity=0 -> lower=-2.75 upper=2.75 effort=100 velocity=5; origin xyz=0 -0.27001 0 rpy=1.5708 -1.5708 0 -> xyz=0 -0.27001 0 rpy=1.5707963  -1.5707963  0
- joint joint6: limit lower=-0.73 upper=0.95 effort=0 velocity=0 -> lower=-0.73 upper=0.95 effort=100 velocity=5; origin xyz=0 0 0 rpy=1.5708 -1.5708 0 -> xyz=0 0 0 rpy=1.5707963  -1.5707963  0
- joint joint7: limit lower=-1.57 upper=1.57 effort=0 velocity=0 -> lower=-1.5707963 upper=1.5707963 effort=100 velocity=5; origin xyz=0 -0.0235 0 rpy=1.5708 0 0 -> xyz=0 -0.0235 0 rpy=1.5707963 0 0
