Commit message: 增加piper lift 案例，训练效果良好

File: src/isaac_so_arm101/robots/piper_description/urdf/piper_description_v100_realsense_camera_v2_dark.urdf (robot description, URDF)
Before this commit: robot piper_camera, 9 links, 8 joints
Joints:
- joint piper_finger_joint7: origin xyz=0 0 0.13503 rpy=1.5708 0 1.5708 -> xyz=0.0 0 0.13503 rpy=1.5708 0 1.5708
- joint piper_finger_joint8: limit lower=-0.05 upper=0 effort=100 velocity=1 -> lower=-0.05 upper=0.00 effort=100 velocity=1; mimic joint=piper_finger_joint8 multiplier=-1 offset=0 -> (none)
